Commit message: added four wheels to the simulation

File: gary_robot_description/gary.urdf (robot description, URDF)
Before this commit: robot gary, 1 links, 0 joints
Links:
- added link left_front_wheel; visual cylinder length=0.058 radius=0.11
- added link left_rear_wheel; visual cylinder length=0.058 radius=0.11
- added link right_front_wheel; visual cylinder length=0.058 radius=0.11
- added link right_rear_wheel; visual cylinder length=0.058 radius=0.11
- link base_link: geometry visual box size=0.4 0.4 0.2
Joints:
- added joint base_lf_wheel_joint: type fixed, parent base_link, child left_front_wheel, origin xyz=0.15 0.229 0.055 rpy=1.5708 0.0 0.0
- added joint base_lr_wheel_joint: type fixed, parent base_link, child left_rear_wheel, origin xyz=-0.15 0.229 0.055 rpy=1.5708 0.0 0.0
- added joint base_rf_wheel_joint: type fixed, parent base_link, child right_front_wheel, origin xyz=0.15 -0.229 0.055 rpy=1.5708 0.0 0.0
- added joint base_rr_wheel_joint: type fixed, parent base_link, child right_rear_wheel, origin xyz=-0.15 -0.229 0.055 rpy=1.5708 0.0 0.0
