Commit message: added launch files both python and xml.

File: gary_robot_description/urdf/gary.urdf (robot description, URDF)
Before this commit: robot gary, 5 links, 4 joints
Links:
- added link base_footprint
Joints:
- added joint base_joint: type fixed, parent base_footprint, child base_link, origin xyz=0 0 0.055 rpy=0 0 0
- joint base_lf_wheel_joint: axis (none) -> 0 1 0; origin xyz=0.15 0.229 0.055 rpy=1.5708 0.0 0.0 -> xyz=0.15 0.229 0.055 rpy=0.0 0.0 0.0; type fixed -> continuous
- joint base_lr_wheel_joint: axis (none) -> 0 1 0; origin xyz=-0.15 0.229 0.055 rpy=1.5708 0.0 0.0 -> xyz=-0.15 0.229 0.055 rpy=0.0 0.0 0.0; type fixed -> continuous
- joint base_rf_wheel_joint: axis (none) -> 0 1 0; origin xyz=0.15 -0.229 0.055 rpy=1.5708 0.0 0.0 -> xyz=0.15 -0.229 0.055 rpy=0.0 0.0 0.0; type fixed -> continuous
- joint base_rr_wheel_joint: axis (none) -> 0 1 0; origin xyz=-0.15 -0.229 0.055 rpy=1.5708 0.0 0.0 -> xyz=-0.15 -0.229 0.055 rpy=0.0 0.0 0.0; type fixed -> continuous
