Commit message: adding meshes

File: gary_robot_description/urdf/mobile_base.xacro (robot description, xacro)
@@ -31,5 +31,14 @@
   <xacro:wheel_link prefix="left_front" />
   <xacro:wheel_link prefix="right_rear" />
-  <xacro:wheel_link prefix="left_rear" />
+  <!-- <xacro:wheel_link prefix="left_rear" /> -->
+  <link name="left_rear_wheel_link">
+      <visual>
+      <geometry>
+          <mesh filename="package://gary_robot_description/meshes/left_tire.stl" scale="0.001 0.001 0.001"/>
+      </geometry>
+      <origin xyz="0 0 0" rpy="0 0 ${pi}"/>
+      <material name="green" />
+      </visual>
+  </link>
   <joint name="base_joint" type="fixed">
     <parent link="base_footprint" />

Commit message: ros jazzy image

File: gary_robot_description/urdf/mobile_base.xacro (robot description, xacro)
@@ -31,14 +31,5 @@
   <xacro:wheel_link prefix="left_front" />
   <xacro:wheel_link prefix="right_rear" />
-  <!-- <xacro:wheel_link prefix="left_rear" /> -->
-  <link name="left_rear_wheel_link">
-      <visual>
-      <geometry>
-          <mesh filename="package://gary_robot_description/meshes/left_tire.stl" scale="0.001 0.001 0.001"/>
-      </geometry>
-      <origin xyz="0 0 0" rpy="0 0 ${pi}"/>
-      <material name="green" />
-      </visual>
-  </link>
+  <xacro:wheel_link prefix="left_rear" />
   <joint name="base_joint" type="fixed">
     <parent link="base_footprint" />
@@ -49,5 +40,5 @@
     <parent link="base_link" />
     <child link="right_front_wheel_link" />
-    <origin xyz="0.15 ${-1*(base_width + wheel_length)/2} ${base_heigh/4}" rpy="0.0 0.0 0.0" />
+    <origin xyz="${base_length/3} ${-1*(base_width + wheel_length)/2} ${base_heigh/4}" rpy="0.0 0.0 0.0" />
     <axis xyz="0 1 0"/>
   </joint>
@@ -55,5 +46,5 @@
     <parent link="base_link" />
     <child link="right_rear_wheel_link" />
-    <origin xyz="-0.15 ${-1*(base_width + wheel_length)/2} ${base_heigh/4}" rpy="0.0 0.0 0.0" />
+    <origin xyz="${-base_length/3} ${-1*(base_width + wheel_length)/2} ${base_heigh/4}" rpy="0.0 0.0 0.0" />
     <axis xyz="0 1 0"/>
   </joint>
@@ -61,5 +52,5 @@
     <parent link="base_link" />
     <child link="left_front_wheel_link" />
-    <origin xyz="0.15 ${(base_width + wheel_length)/2} ${base_heigh/4}" rpy="0.0 0.0 0.0" />
+    <origin xyz="${base_length/3} ${(base_width + wheel_length)/2} ${base_heigh/4}" rpy="0.0 0.0 0.0" />
     <axis xyz="0 1 0"/>
   </joint>
@@ -67,5 +58,5 @@
     <parent link="base_link" />
     <child link="left_rear_wheel_link" />
-    <origin xyz="-0.15 ${(base_width+wheel_length)/2} ${base_heigh/4}" rpy="0.0 0.0 0.0" />
+    <origin xyz="${-base_length/3} ${(base_width+wheel_length)/2} ${base_heigh/4}" rpy="0.0 0.0 0.0" />
     <axis xyz="0 1 0"/>
   </joint>
