Commit message: collition and inertia tags added

File: gary_robot_description/urdf/common_properties.xacro (robot description, xacro)
@@ -10,3 +10,21 @@
     <color rgba="1.0 0 0 1"/>
   </material>
+  <xacro:macro name="box_inertia" params="m x y z o_xyz o_rpy">
+    <inertial>
+      <mass value="${m}" />
+      <origin xyz="${o_xyz}" rpy="${o_rpy}" />
+      <inertia ixx="${(m/12.0)*(y*y + z*z)}" ixy="0.0" ixz="0.0"
+               iyy="${(m/12.0)*(x*x + z*z)}" iyz="0.0"
+               izz="${(m/12.0)*(x*x + y*y)}" />
+    </inertial>
+  </xacro:macro>
+  <xacro:macro name="cylinder_inertia" params="m r h o_xyz o_rpy">
+    <inertial>
+      <mass value="${m}" />
+      <origin xyz="${o_xyz}" rpy="${o_rpy}" />
+      <inertia ixx="${(m/12.0)*(3*r**2.0 + h**2.0)}" ixy="0.0" ixz="0.0"
+               iyy="${(m/12.0)*(3*r**2.0 + h**2.0)}" iyz="0.0"
+               izz="${(m/2.0)*(r**2.0)}" />
+    </inertial>
+  </xacro:macro>
 </robot>

File: gary_robot_description/urdf/mobile_base.xacro (robot description, xacro)
@@ -13,7 +13,14 @@
         <box size="${base_length} ${base_width} ${base_heigh}"/>
       </geometry>
-      <origin xyz="0 0 0.1" rpy="0 0 0"/>
+      <origin xyz="0 0 ${base_heigh/2.0}" rpy="0 0 0"/>
       <material name="blue" />
     </visual>
+    <collision>
+      <origin xyz="0 0 ${base_heigh/2.0}" rpy="0 0 0"/>
+      <geometry>
+        <box size="${base_length} ${base_width} ${base_heigh}"/>
+      </geometry>
+    </collision>
+    <xacro:box_inertia m="10" x="${base_length}" y="${base_width}" z="${base_heigh}" o_xyz="0 0 ${base_heigh/2.0}" o_rpy="0 0 0" />
   </link>
   <xacro:macro name="wheel_link" params="prefix">
@@ -26,4 +33,11 @@
         <material name="green" />
       </visual>
+      <collision>
+        <origin xyz="0 0 0" rpy="${pi/2} 0 0"/>
+        <geometry>
+          <cylinder radius="${wheel_radius}" length="${wheel_length}"/>
+        </geometry>
+      </collision>
+      <xacro:cylinder_inertia m="3.0" r="${wheel_radius}" h="${wheel_length}" o_xyz="0 0 0" o_rpy="${pi/2} 0 0" />
     </link>
   </xacro:macro>
